File: he_sensor.kicad_sch (KiCad schematic)
At the start: 2 parts, among them IC4 CT100LW-IS6

Commit message: [UPDATE](PCB) placed LEDs
Parts:
- renumbered IC4 to TMR1

Commit message: [ADD](PCB) led and tmr caps placement
Parts:
- renumbered C28 to C_TMR7001, TMR1 to TMR7001
