File: RyzzenKeyboard.kicad_sch (KiCad schematic)
At the start: 28 parts, among them IC1 LD39100PU33RY, J1 Conn_01x16_Socket, J2 Conn_01x16_Socket, J3 TC2050, J8 GSB1C4621DS1HR, U1 W25Q32JVSS, U2 STM32F411CEUx, Y1 25MHz

Commit message: [FIX](USB) main usb net labels
Parts:
- renumbered D2 to D1, J8 to J2, J2 to J3, J3 to J4, R6 to R3, R16 to R4
Changed lines of the file:
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@@
 		(dnp no)
 		(fields_autoplaced yes)
-		(property "Reference" "#PWR030"
+		(property "Reference" "#PWR031"
 			(at 151.13 158.75 0)
 			(effects
@@
 			(project "RyzzenKeyboard"
 				(path "/5d44d704-6136-40a8-98a4-93f001ea8743"
-					(reference "#PWR030")
+					(reference "#PWR031")
 					(unit 1)
 				)
@@
 		(dnp no)
 		(fields_autoplaced yes)
-		(property "Reference" "#PWR021"
+		(property "Reference" "#PWR022"
 			(at 137.16 194.31 0)
 			(effects
@@
 			(project "RyzzenKeyboard"
 				(path "/5d44d704-6136-40a8-98a4-93f001ea8743"
-					(reference "#PWR021")
+					(reference "#PWR022")
 					(unit 1)
 				)
@@
 		(dnp no)
 		(fields_autoplaced yes)
-		(property "Reference" "#PWR019"
+		(property "Reference" "#PWR020"
 			(at 137.16 163.83 0)
 			(effects
@@
 			(project "RyzzenKeyboard"
 				(path "/5d44d704-6136-40a8-98a4-93f001ea8743"
-					(reference "#PWR019")
+					(reference "#PWR020")
 					(unit 1)
 				)
@@
 		(dnp no)
 		(fields_autoplaced yes)
-		(property "Reference" "#PWR017"
+		(property "Reference" "#PWR018"
 			(at 127 158.75 0)
 			(effects
@@
 			(project "RyzzenKeyboard"
 				(path "/5d44d704-6136-40a8-98a4-93f001ea8743"
-					(reference "#PWR017")
+					(reference "#PWR018")
 					(unit 1)
 				)
@@
 		(dnp no)
 		(fields_autoplaced yes)
-		(property "Reference" "#PWR038"
+		(property "Reference" "#PWR039"
 			(at 259.08 50.8 0)
 			(effects
@@
 			(project ""
 				(path "/5d44d704-6136-40a8-98a4-93f001ea8743"
-					(reference "#PWR038")
+					(reference "#PWR039")
 					(unit 1)
 				)
@@
 		(on_board yes)
 		(dnp no)
-		(property "Reference" "R16"
+		(property "Reference" "R4"
 			(at 173.99 108.712 90)
 			(effects
@@
 			(project "RyzzenKeyboard"
 				(path "/5d44d704-6136-40a8-98a4-93f001ea8743"
-					(reference "R16")
+					(reference "R4")
 					(unit 1)
 				)
@@
 		(dnp no)
 		(fields_autoplaced yes)
-		(property "Reference" "#PWR036"
+		(property "Reference" "#PWR037"
 			(at 198.12 53.34 0)
 			(effects
@@
 			(project "RyzzenKeyboard"
 				(path "/5d44d704-6136-40a8-98a4-93f001ea8743"
-					(reference "#PWR036")
+					(reference "#PWR037")
 					(unit 1)
 				)
@@
 		(dnp no)
 		(fields_autoplaced yes)
-		(property "Reference" "#PWR020"
+		(property "Reference" "#PWR021"
 			(at 137.16 171.45 0)
 			(effects
@@
 			(project "RyzzenKeyboard"
 				(path "/5d44d704-6136-40a8-98a4-93f001ea8743"
-					(reference "#PWR020")
+					(reference "#PWR021")
 					(unit 1)
 				)
@@
 		(on_board yes)
 		(dnp no)
-		(property "Reference" "#PWR018"
+		(property "Reference" "#PWR019"
 			(at 127 161.29 0)
 			(effects
@@
 			(project "RyzzenKeyboard"
 				(path "/5d44d704-6136-40a8-98a4-93f001ea8743"
-					(reference "#PWR018")
+					(reference "#PWR019")
 					(unit 1)
 				)
@@
 		(on_board yes)
 		(dnp no)
-		(property "Reference" "#PWR079"
+		(property "Reference" "#PWR036"
 			(at 171.45 96.52 0)
 			(effects
@@
 			(project "RyzzenKeyboard"
 				(path "/5d44d704-6136-40a8-98a4-93f001ea8743"
-					(reference "#PWR079")
+					(reference "#PWR036")
 					(unit 1)
 				)
@@
 		(on_board yes)
 		(dnp no)
-		(property "Reference" "#PWR037"
+		(property "Reference" "#PWR038"
 			(at 248.92 55.88 0)
 			(effects
@@
 			(project "RyzzenKeyboard"
 				(path "/5d44d704-6136-40a8-98a4-93f001ea8743"
-					(reference "#PWR037")
+					(reference "#PWR038")
 					(unit 1)
 				)
@@
 		(on_board yes)
 		(dnp no)
-		(property "Reference" "#PWR031"
+		(property "Reference" "#PWR032"
 			(at 151.13 161.29 0)
 			(effects
@@
 			(project "RyzzenKeyboard"
 				(path "/5d44d704-6136-40a8-98a4-93f001ea8743"
-					(reference "#PWR031")
+					(reference "#PWR032")
 					(unit 1)
 				)
@@
 		(on_board yes)
 		(dnp no)
-		(property "Reference" "#PWR025"
+		(property "Reference" "#PWR026"
 			(at 144.78 92.71 0)
 			(effects
@@
 			(project "RyzzenKeyboard"
 				(path "/5d44d704-6136-40a8-98a4-93f001ea8743"
-					(reference "#PWR025")
+					(reference "#PWR026")
 					(unit 1)
 				)
@@
 		(dnp no)
 		(fields_autoplaced yes)
-		(property "Reference" "#PWR034"
+		(property "Reference" "#PWR035"
 			(at 161.29 194.31 0)
 			(effects
@@
 			(project "RyzzenKeyboard"
 				(path "/5d44d704-6136-40a8-98a4-93f001ea8743"
-					(reference "#PWR034")
+					(reference "#PWR035")
 					(unit 1)
 				)
@@
 		(dnp no)
 		(fields_autoplaced yes)
-		(property "Reference" "#PWR016"
+		(property "Reference" "#PWR017"
 			(at 137.16 156.21 0)
 			(effects
@@
 			(project "RyzzenKeyboard"
 				(path "/5d44d704-6136-40a8-98a4-93f001ea8743"
-					(reference "#PWR016")
+					(reference "#PWR017")
 					(unit 1)
 				)
@@
 		(on_board yes)
 		(dnp no)
-		(property "Reference" "D2"
+		(property "Reference" "D1"
 			(at 126.492 108.204 0)
 			(effects
@@
 			(project "RyzzenKeyboard"
 				(path "/5d44d704-6136-40a8-98a4-93f001ea8743"
-					(reference "D2")
+					(reference "D1")
 					(unit 1)
 				)
@@
 		(on_board yes)
 		(dnp no)
-		(property "Reference" "R6"
+		(property "Reference" "R3"
 			(at 128.27 122.428 90)
 			(effects
@@
 			(project "RyzzenKeyboard"
 				(path "/5d44d704-6136-40a8-98a4-93f001ea8743"
-					(reference "R6")
+					(reference "R3")
 					(unit 1)
 				)
@@
 		(dnp no)
 		(fields_autoplaced yes)
-		(property "Reference" "#PWR029"
+		(property "Reference" "#PWR030"
 			(at 161.29 156.21 0)
 			(effects
@@
 			(project "RyzzenKeyboard"
 				(path "/5d44d704-6136-40a8-98a4-93f001ea8743"
-					(reference "#PWR029")
+					(reference "#PWR030")
 					(unit 1)
 				)
@@
 		(dnp no)
 		(fields_autoplaced yes)
-		(property "Reference" "#PWR033"
+		(property "Reference" "#PWR034"
 			(at 161.29 171.45 0)
 			(effects
@@
 			(project "RyzzenKeyboard"
 				(path "/5d44d704-6136-40a8-98a4-93f001ea8743"
-					(reference "#PWR033")
+					(reference "#PWR034")
 					(unit 1)
 				)
@@
 		(dnp no)
 		(fields_autoplaced yes)
-		(property "Reference" "#PWR027"
+		(property "Reference" "#PWR028"
 			(at 147.32 50.8 0)
 			(effects
@@
 			(project "RyzzenKeyboard"
 				(path "/5d44d704-6136-40a8-98a4-93f001ea8743"
-					(reference "#PWR027")
+					(reference "#PWR028")
 					(unit 1)
 				)
@@
 		(dnp no)
 		(fields_autoplaced yes)
-		(property "Reference" "J2"
+		(property "Reference" "J3"
 			(at 150.495 151.13 0)
 			(effects
@@
 			(project "RyzzenKeyboard"
 				(path "/5d44d704-6136-40a8-98a4-93f001ea8743"
-					(reference "J2")
+					(reference "J3")
 					(unit 1)
 				)
@@
 		(dnp no)
 		(fields_autoplaced yes)
-		(property "Reference" "#PWR075"
+		(property "Reference" "#PWR024"
 			(at 138.43 95.25 0)
 			(effects
@@
 			(project "RyzzenKeyboard"
 				(path "/5d44d704-6136-40a8-98a4-93f001ea8743"
-					(reference "#PWR075")
+					(reference "#PWR024")
 					(unit 1)
 				)
@@
 		(dnp no)
 		(fields_autoplaced yes)
-		(property "Reference" "#PWR032"
+		(property "Reference" "#PWR033"
 			(at 161.29 163.83 0)
 			(effects
@@
 			(project "RyzzenKeyboard"
 				(path "/5d44d704-6136-40a8-98a4-93f001ea8743"
-					(reference "#PWR032")
+					(reference "#PWR033")
 					(unit 1)
 				)
@@
 		(on_board yes)
 		(dnp no)
-		(property "Reference" "#PWR026"
+		(property "Reference" "#PWR027"
 			(at 147.32 34.29 0)
 			(effects
@@
 			(project "RyzzenKeyboard"
 				(path "/5d44d704-6136-40a8-98a4-93f001ea8743"
-					(reference "#PWR026")
+					(reference "#PWR027")
 					(unit 1)
 				)
@@
 		(dnp no)
 		(fields_autoplaced yes)
-		(property "Reference" "J3"
+		(property "Reference" "J4"
 			(at 160.02 57.15 0)
 			(effects
@@
 			(project ""
 				(path "/5d44d704-6136-40a8-98a4-93f001ea8743"
-					(reference "J3")
+					(reference "J4")
 					(unit 1)
 				)
@@
 		(on_board yes)
 		(dnp no)
-		(property "Reference" "#PWR028"
+		(property "Reference" "#PWR029"
 			(at 151.13 71.12 0)
 			(effects
@@
 			(project "RyzzenKeyboard"
 				(path "/5d44d704-6136-40a8-98a4-93f001ea8743"
-					(reference "#PWR028")
+					(reference "#PWR029")
 					(unit 1)
 				)
@@
 		(on_board yes)
 		(dnp no)
-		(property "Reference" "#PWR078"
+		(property "Reference" "#PWR016"
 			(at 130.81 132.08 0)
 			(effects
@@
 			(project "RyzzenKeyboard"
 				(path "/5d44d704-6136-40a8-98a4-93f001ea8743"
-					(reference "#PWR078")
+					(reference "#PWR016")
 					(unit 1)
 				)
@@
 		(on_board yes)
 		(dnp no)
-		(property "Reference" "#PWR076"
+		(property "Reference" "#PWR023"
 			(at 133.35 105.41 0)
 			(effects
@@
 			(project "RyzzenKeyboard"
 				(path "/5d44d704-6136-40a8-98a4-93f001ea8743"
-					(reference "#PWR076")
+					(reference "#PWR023")
 					(unit 1)
 				)
@@
 		(dnp no)
 		(fields_autoplaced yes)
-		(property "Reference" "J8"
+		(property "Reference" "J2"
 			(at 154.94 104.14 0)
 			(effects
@@
 			(project ""
 				(path "/5d44d704-6136-40a8-98a4-93f001ea8743"
-					(reference "J8")
+					(reference "J2")
 					(unit 1)
 				)
@@
 		(dnp no)
 		(fields_autoplaced yes)
-		(property "Reference" "#PWR077"
+		(property "Reference" "#PWR025"
 			(at 139.7 142.24 0)
 			(effects
@@
 			(project "RyzzenKeyboard"
 				(path "/5d44d704-6136-40a8-98a4-93f001ea8743"
-					(reference "#PWR077")
+					(reference "#PWR025")
 					(unit 1)
 				)

Commit message: [UPDATE](PCB) placed LEDs
Parts:
- removed Y1: 25MHz, ECS-250-8-30B-CKM:XTAL_ECS-250-8-30B-CKM, symbol Device:Crystal_GND24
- added Y1: ECS-250-8-30B-CKM, ECS-250-8-30B-CKM:XTAL_ECS-250-8-30B-CKM, symbol ECS-250-8-30B-CKM:ECS-250-8-30B-CKM
Connections:
- net GND: now also Y1.2 (GND), Y1.4 (GND)
- net HSE_IN: now also Y1.3 (OUT/IN)
- net HSE_OUT: now also Y1.1 (IN/OUT)

Commit message: [ADD](PCB) led and tmr caps placement
Parts:
- renumbered C1 to C1001, C2 to C1002, C3 to C1003, C4 to C1004, C5 to C1005, C6 to C1006, C7 to C1007, C8 to C1008, C9 to C1009, C10 to C1010, C11 to C1011, C12 to C1012, C13 to C1013, D1 to D1001, FB1 to FB1001, IC1 to IC1001, J1 to J1001, J2 to J1002, J3 to J1003, J4 to J1004, R1 to R1001, R2 to R1002, R3 to R1003, R4 to R1004, R5 to R1005, U1 to U1001, U2 to U1002, Y1 to Y1001

Commit message: [ADD](Mountinghole)
Connections:
- net GND: no longer J1001.10 (Pin_10), J1003.10 (Pin_10)
- net nWR: now also U1002.12 (PA2); no longer U1002.13 (PA3)
- net D2: now reaches U1002.14 (PA4)
- net D2: now also J1003.10 (Pin_10)
- new net D1: J1001.10 (Pin_10), U1002.13 (PA3)
- no-connect marks 12 -> 10
Changed lines of the file:
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@@
 	)
 	(no_connect
-		(at 116.84 63.5)
-	)
-	(no_connect
-		(at 116.84 58.42)
-	)
-	(no_connect
 		(at 116.84 73.66)
 	)
@@
 		)
 	)
+	(label "D2"
+		(at 154.94 171.45 0)
+		(effects
+			(font
+				(size 1.27 1.27)
+			)
+			(justify left bottom)
+		)
+	)
+	(label "D1"
+		(at 130.81 171.45 0)
+		(effects
+			(font
+				(size 1.27 1.27)
+			)
+			(justify left bottom)
+		)
+	)
 	(label "SPI1_MOSI"
 		(at 240.03 125.73 90)
@@
 		)
 	)
+	(label "D1"
+		(at 116.84 60.96 0)
+		(effects
+			(font
+				(size 1.27 1.27)
+			)
+			(justify left bottom)
+		)
+	)
 	(label "A1"
 		(at 130.81 184.15 0)
@@
 		)
 	)
-	(label "nWR"
-		(at 116.84 60.96 0)
+	(label "DA+"
+		(at 116.84 53.34 0)
 		(effects
 			(font
@@
 		)
 	)
-	(label "DA+"
-		(at 116.84 53.34 0)
+	(label "nCS2"
+		(at 130.81 176.53 0)
 		(effects
 			(font
@@
 		)
 	)
-	(label "nCS2"
-		(at 130.81 176.53 0)
+	(label "D2"
+		(at 116.84 63.5 0)
 		(effects
 			(font
@@
 		)
 	)
+	(label "nWR"
+		(at 116.84 58.42 0)
+		(effects
+			(font
+				(size 1.27 1.27)
+			)
+			(justify left bottom)
+		)
+	)
 	(label "SPI1_MISO"
 		(at 31.75 120.65 180)
@@
 	)
 	(symbol
-		(lib_id "power:GND")
-		(at 130.81 171.45 90)
-		(unit 1)
-		(exclude_from_sim no)
-		(in_bom yes)
-		(on_board yes)
-		(dnp no)
-		(fields_autoplaced yes)
-		(property "Reference" "#PWR01021"
-			(at 137.16 171.45 0)
-			(effects
-				(font
-					(size 1.27 1.27)
-				)
-				(hide yes)
-			)
-		)
-		(property "Value" "GND"
-			(at 134.62 171.4499 90)
-			(effects
-				(font
-					(size 1.27 1.27)
-				)
-				(justify right)
-			)
-		)
-		(property "Footprint" ""
-			(at 130.81 171.45 0)
-			(effects
-				(font
-					(size 1.27 1.27)
-				)
-				(hide yes)
-			)
-		)
-		(property "Datasheet" ""
-			(at 130.81 171.45 0)
-			(effects
-				(font
-					(size 1.27 1.27)
-				)
-				(hide yes)
-			)
-		)
-		(property "Description" "Power symbol creates a global label with name \"GND\" , ground"
-			(at 130.81 171.45 0)
-			(effects
-				(font
-					(size 1.27 1.27)
-				)
-				(hide yes)
-			)
-		)
-		(pin "1"
-		)
-		(instances
-			(project "RyzzenKeyboard"
-				(path "/5d44d704-6136-40a8-98a4-93f001ea8743"
-					(reference "#PWR01021")
-					(unit 1)
-				)
-			)
-		)
-	)
-	(symbol
 		(lib_id "Device:C")
 		(at 31.75 38.1 0)
@@
 					(unit 1)
 				)
-			)
-		)
-	)
-	(symbol
-		(lib_id "power:GND")
-		(at 154.94 171.45 90)
-		(unit 1)
-		(exclude_from_sim no)
-		(in_bom yes)
-		(on_board yes)
-		(dnp no)
-		(fields_autoplaced yes)
-		(property "Reference" "#PWR01034"
-			(at 161.29 171.45 0)
-			(effects
-				(font
-					(size 1.27 1.27)
-				)
-				(hide yes)
-			)
-		)
-		(property "Value" "GND"
-			(at 158.75 171.4499 90)
-			(effects
-				(font
-					(size 1.27 1.27)
-				)
-				(justify right)
-			)
-		)
-		(property "Footprint" ""
-			(at 154.94 171.45 0)
-			(effects
-				(font
-					(size 1.27 1.27)
-				)
-				(hide yes)
-			)
-		)
-		(property "Datasheet" ""
-			(at 154.94 171.45 0)
-			(effects
-				(font
-					(size 1.27 1.27)
-				)
-				(hide yes)
-			)
-		)
-		(property "Description" "Power symbol creates a global label with name \"GND\" , ground"
-			(at 154.94 171.45 0)
-			(effects
-				(font
-					(size 1.27 1.27)
-				)
-				(hide yes)
-			)
-		)
-		(pin "1"
-		)
-		(instances
-			(project "RyzzenKeyboard"
-				(path "/5d44d704-6136-40a8-98a4-93f001ea8743"
-					(reference "#PWR01034")
-					(unit 1)
-				)
