File: RyzzenKeyboard.kicad_sch (KiCad schematic)
At the start: 28 parts, among them IC1001 LD39100PU33RY, J1001 Conn_01x16_Socket, J1002 GSB1C4621DS1HR, J1003 Conn_01x16_Socket, J1004 TC2050, U1001 W25Q32JVSS, U1002 STM32F411CEUx, Y1001 ECS-250-8-30B-CKM

Commit message: [ADD](no clue)
Connections:
- net A0: now also U1002.21 (PB10); no longer U1002.18 (PB0)
- net A1: now also U1002.20 (PB2); no longer U1002.19 (PB1)
- net A2: now also U1002.19 (PB1); no longer U1002.20 (PB2)
- net A3: now also U1002.18 (PB0); no longer U1002.21 (PB10)
- net CS_USB1: now also U1002.28 (PB15); no longer U1002.27 (PB14)
- net CS_USB3: now also U1002.27 (PB14); no longer U1002.25 (PB12)
- net VBUS: now also D1001.1 (K), J1002.A4 (VBUS_1), J1002.A9 (VBUS_2)
- net nCS0: now also U1002.42 (PB6); no longer U1002.39 (PB3)
- net nCS1: now also U1002.41 (PB5); no longer U1002.40 (PB4)
- net nCS2: now also U1002.45 (PB8); no longer U1002.41 (PB5)
- net nCS3: now also U1002.43 (PB7); no longer U1002.42 (PB6)
- net nCS4: now also U1002.40 (PB4); no longer U1002.43 (PB7)
- net nCS5: now also U1002.39 (PB3); no longer U1002.45 (PB8)
- net nCS_FLASH: now also U1002.25 (PB12); no longer U1002.28 (PB15)
Changed lines of the file:
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@@
 		)
 	)
-	(label "nCS1"
+	(label "nCS4"
 		(at 81.28 91.44 180)
 		(effects
@@
 		)
 	)
-	(label "A2"
+	(label "A1"
 		(at 81.28 86.36 180)
 		(effects
@@
 		)
 	)
+	(label "VBUS"
+		(at 133.35 114.3 90)
+		(effects
+			(font
+				(size 1.27 1.27)
+			)
+			(justify left bottom)
+		)
+	)
 	(label "nCS0"
 		(at 53.34 176.53 0)
@@
 		)
 	)
-	(label "nCS5"
+	(label "nCS2"
 		(at 81.28 101.6 180)
 		(effects
@@
 		)
 	)
+	(label "CS_USB3"
+		(at 81.28 114.3 180)
+		(effects
+			(font
+				(size 1.27 1.27)
+			)
+			(justify right bottom)
+		)
+	)
 	(label "DA+"
 		(at 116.84 53.34 0)
@@
 		)
 	)
-	(label "nCS_FLASH"
-		(at 81.28 116.84 180)
-		(effects
-			(font
-				(size 1.27 1.27)
-			)
-			(justify right bottom)
-		)
-	)
 	(label "NRST"
 		(at 266.7 148.59 270)
@@
 		)
 	)
-	(label "CS_USB1"
-		(at 81.28 114.3 180)
-		(effects
-			(font
-				(size 1.27 1.27)
-			)
-			(justify right bottom)
-		)
-	)
 	(label "SWDIO"
 		(at 261.62 148.59 270)
@@
 		)
 	)
-	(label "nCS4"
+	(label "nCS3"
 		(at 81.28 99.06 180)
 		(effects
@@
 		)
 	)
+	(label "CS_USB1"
+		(at 81.28 116.84 180)
+		(effects
+			(font
+				(size 1.27 1.27)
+			)
+			(justify right bottom)
+		)
+	)
 	(label "USB+"
 		(at 170.18 114.3 0)
@@
 		)
 	)
-	(label "nCS0"
+	(label "nCS5"
 		(at 81.28 88.9 180)
 		(effects
@@
 		)
 	)
-	(label "nCS2"
+	(label "nCS1"
 		(at 81.28 93.98 180)
-		(effects
-			(font
-				(size 1.27 1.27)
-			)
-			(justify right bottom)
-		)
-	)
-	(label "CS_USB3"
-		(at 81.28 109.22 180)
 		(effects
 			(font
@@
 		)
 	)
-	(label "A3"
+	(label "A0"
 		(at 81.28 106.68 180)
 		(effects
@@
 		)
 	)
-	(label "A0"
+	(label "A3"
 		(at 81.28 81.28 180)
 		(effects
@@
 		)
 	)
-	(label "A1"
+	(label "A2"
 		(at 81.28 83.82 180)
 		(effects
@@
 		)
 	)
-	(label "nCS3"
+	(label "nCS0"
 		(at 81.28 96.52 180)
 		(effects
 			(font
+				(size 1.27 1.27)
+			)
+			(justify right bottom)
+		)
+	)
+	(label "nCS_FLASH"
+		(at 81.28 109.22 180)
+		(effects
+			(font
