File: RyzzenKeyboard.kicad_pcb (KiCad board)
At the start: 2 copper layers, 3.6 x 3.3 mm, 239 parts, among them IC1 LD39100PU33RY, IC10 CT100LW-IS6, IC11 CT100LW-IS6, IC12 CT100LW-IS6, IC13 CT100LW-IS6, IC14 CT100LW-IS6, IC15 CT100LW-IS6, IC16 CT100LW-IS6, IC17 CT100LW-IS6, IC18 CT100LW-IS6, IC19 ADG726BSUZ, IC2 ADG726BSUZ, IC20 CT100LW-IS6, IC21 CT100LW-IS6, IC22 CT100LW-IS6, IC23 CT100LW-IS6, IC24 CT100LW-IS6, IC25 CT100LW-IS6, IC26 CT100LW-IS6, IC27 CT100LW-IS6, IC28 CT100LW-IS6, IC29 CT100LW-IS6, IC3 CT100LW-IS6, IC30 CT100LW-IS6, IC31 CT100LW-IS6, IC32 CT100LW-IS6, IC33 CT100LW-IS6, IC34 CT100LW-IS6, IC35 CT100LW-IS6, IC36 SN74AHCT1G125DBVR, IC4 CT100LW-IS6, IC5 CT100LW-IS6, IC6 CT100LW-IS6, IC7 CT100LW-IS6, IC8 CT100LW-IS6, IC9 CT100LW-IS6, J1 Conn_01x16_Socket, J2 Conn_01x16_Socket, J3 TC2050, J4 GSB1C4621DS1HR, J5 GSB1C4621DS1HR, J6 GSB1C4621DS1HR, J8 GSB1C4621DS1HR, U1 W25Q32JVSS, U2 STM32F411CEUx, U3 STM32F042K4Tx, U36 STM32F042K4Tx, U37 STM32F042K4Tx, Y1 25MHz

Commit message: [FIX](USB) main usb net labels
Parts:
- moved C1 191.2 mm to (-101.6, 95.8)
- moved C10 191.2 mm to (-97.2, 100.8)
- moved C100 191.2 mm to (-143.6, 77.0)
- moved C101 191.2 mm to (-132.6, 115.6)
- moved C102 191.2 mm to (-121.5, 89.8)
- moved C103 191.2 mm to (-154.7, 89.8)
- moved C104 191.2 mm to (-37.4, 39.9)
- moved C11 191.2 mm to (-97.2, 103.3)
- moved C12 191.2 mm to (-97.2, 105.8)
- moved C13 191.2 mm to (-97.2, 108.3)
- moved C14 191.2 mm to (-101.6, 118.0)
- moved C15 191.2 mm to (-101.6, 120.5)
- moved C16 191.2 mm to (-101.6, 123.0)
- moved C17 191.2 mm to (-101.6, 125.5)
- moved C18 191.2 mm to (-101.6, 128.0)
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- renumbered C21 to C20, C22 to C21, C70 to C22, C71 to C23, C72 to C24, C73 to C25, C74 to C26, C20 to C27, C23 to C28, C24 to C29, C25 to C30, C26 to C31, C27 to C32, C28 to C33, C29 to C34, C30 to C35, C31 to C36, C32 to C37, C33 to C38, C34 to C39, C35 to C40, C36 to C41, C37 to C42, C38 to C43, C39 to C44, C40 to C45, C41 to C46, C42 to C47, C43 to C48, C44 to C49, C45 to C50, C46 to C51, C47 to C52, C48 to C53, C49 to C54, C50 to C55, C51 to C56, C52 to C57, C53 to C58, C54 to C59, C55 to C60, C56 to C61, C57 to C62, C64 to C63, C65 to C64, C66 to C65, C67 to C66, C68 to C67, C69 to C68, C75 to C69, C76 to C70, C77 to C71, C78 to C72, C79 to C73, C80 to C74, C81 to C75, C82 to C76, C83 to C77, C84 to C78, C85 to C79, C86 to C80, C58 to C81, C59 to C82, C60 to C83, C61 to C84, C62 to C85, C63 to C86, D2 to D1, D12 to D10, D13 to D11, D14 to D12, D15 to D13, D16 to D14, D17 to D15, D18 to D16, D19 to D17, D6 to D18, D20 to D19, D1 to D2, D21 to D20, D22 to D21, D23 to D22, D24 to D23, D25 to D24, D26 to D25, D27 to D26, D28 to D27, D29 to D28, D30 to D29, D4 to D3, D31 to D30, D32 to D31, D33 to D32, D34 to D33, D35 to D34, D36 to D35, D37 to D36, D5 to D4, D3 to D5, D8 to D6, D9 to D7, D10 to D8, D11 to D9, FB4 to FB3, FB3 to FB4, IC9 to IC10, IC10 to IC11, IC11 to IC12, IC12 to IC13, IC13 to IC14, IC14 to IC15, IC15 to IC16, IC16 to IC17, IC17 to IC18, IC18 to IC19, IC19 to IC20, IC20 to IC21, IC21 to IC22, IC22 to IC23, IC23 to IC24, IC24 to IC25, IC25 to IC26, IC26 to IC27, IC27 to IC28, IC28 to IC29, IC36 to IC3, IC29 to IC30, IC30 to IC31, IC31 to IC32, IC32 to IC33, IC33 to IC34, IC34 to IC35, IC35 to IC36, IC3 to IC4, IC4 to IC5, IC5 to IC6, IC6 to IC7, IC7 to IC8, IC8 to IC9, J8 to J2, J2 to J3, J3 to J4, J4 to J5, J5 to J6, J6 to J7, R8 to R11, R7 to R12, R12 to R13, R11 to R14, R6 to R3, R16 to R4, R4 to R6, R3 to R7, R9 to R8, R15 to R9, U4 to ST1, U13 to ST10, U14 to ST11, U15 to ST12, U16 to ST13, U17 to ST14, U18 to ST15, U19 to ST16, U20 to ST17, U21 to ST18, U22 to ST19, U5 to ST2, U23 to ST20, U24 to ST21, U25 to ST22, U26 to ST23, U27 to ST24, U28 to ST25, U29 to ST26, U30 to ST27, U31 to ST28, U32 to ST29, U6 to ST3, U33 to ST30, U34 to ST31, U35 to ST32, U7 to ST4, U8 to ST5, U9 to ST6, U10 to ST7, U11 to ST8, U12 to ST9, U37 to U4, U36 to U5
Other:
- copper layers 2 -> 4

Commit message: [ADD](PCB) outlines
Parts:
- moved ST1 220.5 mm to (57.1, -38.1)
Other:
- board size 3.6 x 3.3 mm -> 244.1 x 133.4 mm

Commit message: [UPDATE](PCB) placed LEDs
Parts:
- removed D6: SK6812MINI-E, kicad-keyboard-parts:MX_SK6812MINI-E_REV
- removed IC10, IC11, IC12, IC14, IC15, IC16, IC17, IC18, IC19, IC21, IC22, IC23, IC24, IC25, IC26, IC27, IC28, IC29, IC30, IC31, IC32, IC33, IC34, IC35, IC36, IC5, IC6, IC7, IC8, IC9: CT100LW-IS6, CT100LW-IS6:SOT95P280X135-6N
- removed IC20: ADG726BSUZ, ADG726BSUZ:QFP50P900X900X120-48N
- removed ST1, ST10, ST11, ST12, ST13, ST14, ST15, ST16, ST17, ST18, ST19, ST2, ST20, ST21, ST22, ST23, ST24, ST25, ST26, ST27, ST28, ST29, ST3, ST30, ST31, ST32, ST4, ST5, ST6, ST7, ST8, ST9: ~, Switch_Keyboard_Cherry_MX:SW_Cherry_MX_PCB_Mag_1.00u
- added C28: 100nF, Capacitor_SMD:C_0603_1608Metric_Pad1.08x0.95mm_HandSolder, F.Cu at (-71.5, 168.9)
- added C29: 100nF, Capacitor_SMD:C_0603_1608Metric_Pad1.08x0.95mm_HandSolder, F.Cu at (-92.4, 164.3)
- added C30: 10uF, Capacitor_SMD:C_0603_1608Metric_Pad1.08x0.95mm_HandSolder, F.Cu at (-92.4, 166.8)
- added C31: 100nF, Capacitor_SMD:C_0603_1608Metric_Pad1.08x0.95mm_HandSolder, F.Cu at (-78.8, 168.9)
- added C32: 100nF, Capacitor_SMD:C_0603_1608Metric_Pad1.08x0.95mm_HandSolder, F.Cu at (-89.3, 200.5)
- added C33: 100nF, Capacitor_SMD:C_0603_1608Metric_Pad1.08x0.95mm_HandSolder, F.Cu at (-67.4, 182.4)
- added C34: 100nF, Capacitor_SMD:C_0603_1608Metric_Pad1.08x0.95mm_HandSolder, F.Cu at (-82.0, 182.4)
- added C35: 100nF, Capacitor_SMD:C_0603_1608Metric_Pad1.08x0.95mm_HandSolder, F.Cu at (-96.6, 200.5)
- added C36: 100nF, Capacitor_SMD:C_0603_1608Metric_Pad1.08x0.95mm_HandSolder, F.Cu at (-89.3, 182.4)
- added C37: 100nF, Capacitor_SMD:C_0603_1608Metric_Pad1.08x0.95mm_HandSolder, F.Cu at (-103.9, 209.6)
- added C38: 100nF, Capacitor_SMD:C_0603_1608Metric_Pad1.08x0.95mm_HandSolder, F.Cu at (-96.6, 209.6)
- added C39: 100nF, Capacitor_SMD:C_0603_1608Metric_Pad1.08x0.95mm_HandSolder, F.Cu at (-82.0, 191.4)
- added C40: 100nF, Capacitor_SMD:C_0603_1608Metric_Pad1.08x0.95mm_HandSolder, F.Cu at (-67.4, 191.4)
- added C41: 100nF, Capacitor_SMD:C_0603_1608Metric_Pad1.08x0.95mm_HandSolder, F.Cu at (-82.0, 200.5)
- added C42: 100nF, Capacitor_SMD:C_0603_1608Metric_Pad1.08x0.95mm_HandSolder, F.Cu at (-60.1, 200.5)
- added C43: 100nF, Capacitor_SMD:C_0603_1608Metric_Pad1.08x0.95mm_HandSolder, F.Cu at (-103.9, 182.4)
- added C44: 100nF, Capacitor_SMD:C_0603_1608Metric_Pad1.08x0.95mm_HandSolder, F.Cu at (-86.1, 168.9)
- added C45: 100nF, Capacitor_SMD:C_0603_1608Metric_Pad1.08x0.95mm_HandSolder, F.Cu at (-103.9, 200.5)
- added C46: 100nF, Capacitor_SMD:C_0603_1608Metric_Pad1.08x0.95mm_HandSolder, F.Cu at (-64.2, 168.9)
- added C47: 100nF, Capacitor_SMD:C_0603_1608Metric_Pad1.08x0.95mm_HandSolder, F.Cu at (-89.3, 191.4)
- added C48: 100nF, Capacitor_SMD:C_0603_1608Metric_Pad1.08x0.95mm_HandSolder, F.Cu at (-89.3, 209.6)
- added C49: 100nF, Capacitor_SMD:C_0603_1608Metric_Pad1.08x0.95mm_HandSolder, F.Cu at (-103.9, 191.4)
- added C50: 100nF, Capacitor_SMD:C_0603_1608Metric_Pad1.08x0.95mm_HandSolder, F.Cu at (-96.6, 191.4)
- added C51: 100nF, Capacitor_SMD:C_0603_1608Metric_Pad1.08x0.95mm_HandSolder, F.Cu at (-67.4, 209.6)
- added C52: 100nF, Capacitor_SMD:C_0603_1608Metric_Pad1.08x0.95mm_HandSolder, F.Cu at (-74.7, 191.4)
- added C53: 100nF, Capacitor_SMD:C_0603_1608Metric_Pad1.08x0.95mm_HandSolder, F.Cu at (-60.1, 182.4)
- added C54: 100nF, Capacitor_SMD:C_0603_1608Metric_Pad1.08x0.95mm_HandSolder, F.Cu at (-74.7, 209.6)
- added C56: 100nF, Capacitor_SMD:C_0603_1608Metric_Pad1.08x0.95mm_HandSolder, F.Cu at (-60.1, 191.4)
- added C57: 100nF, Capacitor_SMD:C_0603_1608Metric_Pad1.08x0.95mm_HandSolder, F.Cu at (-67.4, 200.5)
- added C58: 100nF, Capacitor_SMD:C_0603_1608Metric_Pad1.08x0.95mm_HandSolder, F.Cu at (-96.6, 182.4)
- added C59: 100nF, Capacitor_SMD:C_0603_1608Metric_Pad1.08x0.95mm_HandSolder, F.Cu at (-74.7, 182.4)
- added C60: 100nF, Capacitor_SMD:C_0603_1608Metric_Pad1.08x0.95mm_HandSolder, F.Cu at (-74.7, 200.5)
- added C61: 100nF, Capacitor_SMD:C_0603_1608Metric_Pad1.08x0.95mm_HandSolder, F.Cu at (-82.0, 209.6)
- added IC4: ADG726BSUZ, ADG726BSUZ:QFP50P900X900X120-48N, F.Cu at (-100.3, 168.8)
- added LED3: SK6812MINI-E, kicad-keyboard-parts:MX_SK6812MINI-E_REV, B.Cu at (60.8, 69.8)
- added R10: 10K, Resistor_SMD:R_0603_1608Metric_Pad0.98x0.95mm_HandSolder, F.Cu at (-92.4, 169.3)
- added SWITCH1: , SW_Cherry_MX_PCB_Mag_1.00u, B.Cu at (60.8, 107.9)
- added SWITCH10: , SW_Cherry_MX_PCB_Mag_1.00u, B.Cu at (117.8, 90.9)
- added SWITCH11: , SW_Cherry_MX_PCB_Mag_1.00u, B.Cu at (117.8, 71.9)
- added SWITCH12: , SW_Cherry_MX_PCB_Mag_1.00u, B.Cu at (117.8, 52.8)
- added SWITCH13: , SW_Cherry_MX_PCB_Mag_1.00u, B.Cu at (136.8, 94.9)
- added SWITCH14: , SW_Cherry_MX_PCB_Mag_1.00u, B.Cu at (136.8, 75.9)
- added SWITCH15: , SW_Cherry_MX_PCB_Mag_1.00u, B.Cu at (136.8, 56.8)
- added SWITCH16: , SW_Cherry_MX_PCB_Mag_1.00u, B.Cu at (155.8, 133.0)
- added SWITCH17: , SW_Cherry_MX_PCB_Mag_1.00u, B.Cu at (231.8, 107.9)
- added SWITCH18: , SW_Cherry_MX_PCB_Mag_1.00u, B.Cu at (231.8, 88.9)
- added SWITCH19: , SW_Cherry_MX_PCB_Mag_1.00u, B.Cu at (231.8, 69.8)
- added SWITCH2: , SW_Cherry_MX_PCB_Mag_1.00u, B.Cu at (60.8, 88.9)
- added SWITCH20: , SW_Cherry_MX_PCB_Mag_1.00u, B.Cu at (212.8, 93.9)
- added SWITCH21: , SW_Cherry_MX_PCB_Mag_1.00u, B.Cu at (212.8, 74.9)
- added SWITCH22: , SW_Cherry_MX_PCB_Mag_1.00u, B.Cu at (212.8, 55.8)
- added SWITCH23: , SW_Cherry_MX_PCB_Mag_1.00u, B.Cu at (193.8, 83.9)
- added SWITCH24: , SW_Cherry_MX_PCB_Mag_1.00u, B.Cu at (193.8, 64.9)
- added SWITCH25: , SW_Cherry_MX_PCB_Mag_1.00u, B.Cu at (193.8, 45.8)
- added SWITCH26: , SW_Cherry_MX_PCB_Mag_1.00u, B.Cu at (174.8, 90.9)
- added SWITCH27: , SW_Cherry_MX_PCB_Mag_1.00u, B.Cu at (174.8, 71.9)
- added SWITCH28: , SW_Cherry_MX_PCB_Mag_1.00u, B.Cu at (174.8, 52.8)
- added SWITCH29: , SW_Cherry_MX_PCB_Mag_1.00u, B.Cu at (155.8, 94.9)
- added SWITCH3: , SW_Cherry_MX_PCB_Mag_1.00u, B.Cu at (60.8, 69.8)
- added SWITCH30: , SW_Cherry_MX_PCB_Mag_1.00u, B.Cu at (155.8, 75.9)
- added SWITCH31: , SW_Cherry_MX_PCB_Mag_1.00u, B.Cu at (155.8, 56.8)
- added SWITCH32: , SW_Cherry_MX_PCB_Mag_1.00u, B.Cu at (136.8, 133.0)
- added SWITCH4: , SW_Cherry_MX_PCB_Mag_1.00u, B.Cu at (79.8, 93.9)
- added SWITCH5: , SW_Cherry_MX_PCB_Mag_1.00u, B.Cu at (79.8, 74.9)
- added SWITCH6: , SW_Cherry_MX_PCB_Mag_1.00u, B.Cu at (79.8, 55.8)
- added SWITCH7: , SW_Cherry_MX_PCB_Mag_1.00u, B.Cu at (98.8, 83.9)
- added SWITCH8: , SW_Cherry_MX_PCB_Mag_1.00u, B.Cu at (98.8, 64.9)
- added SWITCH9: , SW_Cherry_MX_PCB_Mag_1.00u, B.Cu at (98.8, 45.8)
- added TMR1: CT100LW-IS6, CT100LW-IS6:SOT95P280X135-6N, F.Cu at (-71.0, 165.3)
- added TMR10: CT100LW-IS6, CT100LW-IS6:SOT95P280X135-6N, F.Cu at (-81.5, 187.9)
- added TMR11: CT100LW-IS6, CT100LW-IS6:SOT95P280X135-6N, F.Cu at (-66.9, 187.9)
- added TMR12: CT100LW-IS6, CT100LW-IS6:SOT95P280X135-6N, F.Cu at (-81.5, 197.0)
- added TMR13: CT100LW-IS6, CT100LW-IS6:SOT95P280X135-6N, F.Cu at (-59.6, 197.0)
- added TMR14: CT100LW-IS6, CT100LW-IS6:SOT95P280X135-6N, F.Cu at (-103.4, 178.8)
- added TMR15: CT100LW-IS6, CT100LW-IS6:SOT95P280X135-6N, F.Cu at (-85.6, 165.3)
- added TMR16: CT100LW-IS6, CT100LW-IS6:SOT95P280X135-6N, F.Cu at (-103.4, 197.0)
- added TMR17: CT100LW-IS6, CT100LW-IS6:SOT95P280X135-6N, F.Cu at (-63.7, 165.3)
- added TMR18: CT100LW-IS6, CT100LW-IS6:SOT95P280X135-6N, F.Cu at (-88.8, 187.9)
- added TMR19: CT100LW-IS6, CT100LW-IS6:SOT95P280X135-6N, F.Cu at (-88.8, 206.0)
- added TMR2: CT100LW-IS6, CT100LW-IS6:SOT95P280X135-6N, F.Cu at (-78.3, 165.3)
- added TMR20: CT100LW-IS6, CT100LW-IS6:SOT95P280X135-6N, F.Cu at (-103.4, 187.9)
- added TMR21: CT100LW-IS6, CT100LW-IS6:SOT95P280X135-6N, F.Cu at (-96.1, 187.9)
- added TMR22: CT100LW-IS6, CT100LW-IS6:SOT95P280X135-6N, F.Cu at (-66.9, 206.0)
- added TMR23: CT100LW-IS6, CT100LW-IS6:SOT95P280X135-6N, F.Cu at (-74.2, 187.9)
- added TMR24: CT100LW-IS6, CT100LW-IS6:SOT95P280X135-6N, F.Cu at (-59.6, 178.8)
- added TMR25: CT100LW-IS6, CT100LW-IS6:SOT95P280X135-6N, F.Cu at (-74.2, 206.0)
- added TMR27: CT100LW-IS6, CT100LW-IS6:SOT95P280X135-6N, F.Cu at (-59.6, 187.9)
- added TMR28: CT100LW-IS6, CT100LW-IS6:SOT95P280X135-6N, F.Cu at (-66.9, 197.0)
- added TMR29: CT100LW-IS6, CT100LW-IS6:SOT95P280X135-6N, F.Cu at (-96.1, 178.8)
- added TMR3: CT100LW-IS6, CT100LW-IS6:SOT95P280X135-6N, F.Cu at (-88.8, 197.0)
- added TMR30: CT100LW-IS6, CT100LW-IS6:SOT95P280X135-6N, F.Cu at (-74.2, 178.8)
- added TMR31: CT100LW-IS6, CT100LW-IS6:SOT95P280X135-6N, F.Cu at (-74.2, 197.0)
- added TMR32: CT100LW-IS6, CT100LW-IS6:SOT95P280X135-6N, F.Cu at (-81.5, 206.0)
- added TMR4: CT100LW-IS6, CT100LW-IS6:SOT95P280X135-6N, F.Cu at (-66.9, 178.8)
- added TMR5: CT100LW-IS6, CT100LW-IS6:SOT95P280X135-6N, F.Cu at (-81.5, 178.8)
- added TMR6: CT100LW-IS6, CT100LW-IS6:SOT95P280X135-6N, F.Cu at (-96.1, 197.0)
- added TMR7: CT100LW-IS6, CT100LW-IS6:SOT95P280X135-6N, F.Cu at (-88.8, 178.8)
- added TMR8: CT100LW-IS6, CT100LW-IS6:SOT95P280X135-6N, F.Cu at (-103.4, 206.0)
- added TMR9: CT100LW-IS6, CT100LW-IS6:SOT95P280X135-6N, F.Cu at (-96.1, 206.0)
- C30: value 100nF -> 10uF
- C45: value 10uF -> 100nF
- IC4: value CT100LW-IS6 -> ADG726BSUZ; footprint CT100LW-IS6:SOT95P280X135-6N -> ADG726BSUZ:QFP50P900X900X120-48N
- LED1: renamed from D3; moved to B.Cu
- LED10: renamed from D13; moved to B.Cu
- LED11: renamed from D14; moved to B.Cu
- LED12: renamed from D15; moved to B.Cu
- LED13: renamed from D16; moved to B.Cu
- LED14: renamed from D17; moved to B.Cu
- LED15: renamed from D19; moved to B.Cu
- LED16: renamed from D20; moved to B.Cu
- LED17: renamed from D21; moved to B.Cu
- LED18: renamed from D22; moved to B.Cu
- LED19: renamed from D23; moved to B.Cu
- LED2: renamed from D4; moved to B.Cu
- LED20: renamed from D24; moved to B.Cu
- LED21: renamed from D25; moved to B.Cu
- LED22: renamed from D26; moved to B.Cu
- LED23: renamed from D27; moved to B.Cu
- LED24: renamed from D28; moved to B.Cu
- LED25: renamed from D29; moved to B.Cu
- LED26: renamed from D30; moved to B.Cu
- LED27: renamed from D31; moved to B.Cu
- LED28: renamed from D32; moved to B.Cu
- LED29: renamed from D33; moved to B.Cu
- LED30: renamed from D34; moved to B.Cu
- LED31: renamed from D35; moved to B.Cu
- LED32: renamed from D36; moved to B.Cu
- LED4: renamed from D7; moved to B.Cu
- LED5: renamed from D8; moved to B.Cu
- LED6: renamed from D9; moved to B.Cu
- LED7: renamed from D10; moved to B.Cu
- LED8: renamed from D11; moved to B.Cu
- LED9: renamed from D12; moved to B.Cu
- Y1: value 25MHz -> ECS-250-8-30B-CKM
- moved LED17 386.0 mm to (231.8, 107.9)
- moved LED22 379.4 mm to (212.8, 55.8)
- moved LED18 361.9 mm to (231.8, 88.9)
- moved LED21 356.7 mm to (212.8, 74.9)
- moved LED25 349.3 mm to (193.8, 45.8)
- moved LED26 328.2 mm to (174.8, 90.9)
- moved LED24 325.1 mm to (193.8, 64.9)
- moved LED16 323.2 mm to (155.8, 133.0)
- moved LED28 316.2 mm to (174.8, 52.8)
- moved LED23 313.1 mm to (193.8, 83.9)
- moved LED31 308.9 mm to (155.8, 56.8)
- moved LED13 301.0 mm to (136.8, 94.9)
- moved LED29 286.0 mm to (155.8, 94.9)
- moved LED10 281.0 mm to (117.8, 90.9)
- moved LED14 279.5 mm to (136.8, 75.9)
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- renumbered C37 to C55, C81 to C80, C82 to C81, C83 to C82, C84 to C83, C80 to C84, D5 to D3, D18 to D4, IC13 to TMR26
Connections:
- IC4 pad 1: /keys/key_bank2/S8A -> /keys/key_bank3/S12A
- IC4 pad 2: unconnected-(IC4-N/C_1-Pad2) -> /keys/key_bank3/S11A
- IC4 pad 3: /keys/key_bank2/S8B -> /keys/key_bank3/S10A
- IC4 pad 4: GND -> /keys/key_bank3/S9A
- IC4 pad 5: unconnected-(IC4-N/C_2-Pad5) -> /keys/key_bank3/S8A
- IC4 pad 6: +3.3VA -> /keys/key_bank3/S7A
- R10 pad 1: Net-(IC20-~{CSA}) -> Net-(IC4-~{CSA})
- Y1 pad 1: /HSE_IN -> /HSE_OUT
- Y1 pad 3: /HSE_OUT -> /HSE_IN
Other:
- outline, holes or cut-outs redrawn

Commit message: [ADD](PCB) led and tmr caps placement
Parts:
- removed C1, C21, C23, C24, C25, C26, C30 (x2): 10uF, Capacitor_SMD:C_0603_1608Metric_Pad1.08x0.95mm_HandSolder
- removed C10, C100, C101, C102, C103, C104, C15, C16, C17, C2, C20, C22, C27, C28 (x2), C29 (x2), C31 (x2), C32 (x2), C33 (x2), C34 (x2), C35 (x2), C36 (x2), C37, C38 (x2), C39 (x2), C4, C40 (x2), C41 (x2), C42 (x2), C43 (x2), C44 (x2), C45 (x2), C46 (x2), C47 (x2), C48 (x2), C49 (x2), C5, C50 (x2), C51 (x2), C52 (x2), C53 (x2), C54 (x2), C55 (x2), C56 (x2), C57 (x2), C58 (x2), C59 (x2), C60 (x2), C61 (x2), C62, C64, C65, C66, C69, C7, C70, C71, C72, C73, C74, C75, C76, C77, C78, C79, C8, C81, C82, C83, C84, C87, C88, C89, C9, C90, C91, C92, C93, C94, C95, C96, C97, C98, C99: 100nF, Capacitor_SMD:C_0603_1608Metric_Pad1.08x0.95mm_HandSolder
- removed C11, C12, C13, C19, C68, C86: 1uF, Capacitor_SMD:C_0603_1608Metric_Pad1.08x0.95mm_HandSolder
- removed C14, C63, C80: 4.7nF, Capacitor_SMD:C_0603_1608Metric_Pad1.08x0.95mm_HandSolder
- removed C18, C67, C85: 10nF, Capacitor_SMD:C_0603_1608Metric_Pad1.08x0.95mm_HandSolder
- removed C3, C6: 6pF, Capacitor_SMD:C_0603_1608Metric_Pad1.08x0.95mm_HandSolder
- removed D1, D2, D3, D4: D_Schottky, CUHS20S30:CUHS20S40H3F
- removed FB1, FB2, FB3, FB4: 120R, BLM21PG121SN1D:BLM21AG102BH1J
- removed IC1: LD39100PU33RY, LD39100PU33RY:SON95P300X300X90-7N-D
- removed IC2, IC4 (x2): ADG726BSUZ, ADG726BSUZ:QFP50P900X900X120-48N
- removed IC3: SN74AHCT1G125DBVR, SN74AHCT1G125DBVR:SOT95P280X145-5N
- removed J1, J3: Conn_01x16_Socket, Connector_JST:JST_XH_S16B-XH-A_1x16_P2.50mm_Horizontal
- removed J2, J5, J6, J7: GSB1C4621DS1HR, GSB1C4621DS1HR:GSB1C4621DS1HR
- removed J4: TC2050, Connector:Tag-Connect_TC2050-IDC-NL_2x05_P1.27mm_Vertical
- removed LED1, LED10, LED11, LED12, LED13, LED14, LED15, LED16, LED17, LED18, LED19, LED2, LED20, LED21, LED22, LED23, LED24, LED25, LED26, LED27, LED28, LED29, LED3, LED30, LED31, LED32, LED4, LED5, LED6, LED7, LED8, LED9: SK6812MINI-E, kicad-keyboard-parts:MX_SK6812MINI-E_REV
- removed R1, R2, R5: 10k, Resistor_SMD:R_0603_1608Metric_Pad0.98x0.95mm_HandSolder
- removed R10 (x2), R8: 10K, Resistor_SMD:R_0603_1608Metric_Pad0.98x0.95mm_HandSolder
- removed R11, R12, R13, R14, R3, R4, R6, R7: 5.1k, Resistor_SMD:R_0603_1608Metric_Pad0.98x0.95mm_HandSolder
- removed R9: 500, Resistor_SMD:R_0603_1608Metric_Pad0.98x0.95mm_HandSolder
- removed TMR1, TMR10, TMR11, TMR12, TMR13, TMR14, TMR15, TMR16, TMR17, TMR18, TMR19, TMR2, TMR20, TMR21, TMR22, TMR23, TMR24, TMR25, TMR26, TMR27, TMR28, TMR29, TMR3, TMR30, TMR31, TMR32, TMR4, TMR5, TMR6, TMR7, TMR8, TMR9: CT100LW-IS6, CT100LW-IS6:SOT95P280X135-6N
- removed U1: W25Q32JVSS, Package_SO:SOIC-8_5.3x5.3mm_P1.27mm
- removed U2: STM32F411CEUx, Package_DFN_QFN:QFN-48-1EP_7x7mm_P0.5mm_EP5.6x5.6mm
- removed U3, U4, U5: STM32F042K4Tx, Package_QFP:LQFP-32_7x7mm_P0.8mm
- removed Y1: ECS-250-8-30B-CKM, ECS-250-8-30B-CKM:XTAL_ECS-250-8-30B-CKM
- added C1001: 10uF, Capacitor_SMD:C_0603_1608Metric_Pad1.08x0.95mm_HandSolder, F.Cu at (-220.5, 73.1)
- added C1002: 100nF, Capacitor_SMD:C_0603_1608Metric_Pad1.08x0.95mm_HandSolder, F.Cu at (-220.5, 75.6)
- added C1003: 6pF, Capacitor_SMD:C_0603_1608Metric_Pad1.08x0.95mm_HandSolder, F.Cu at (-220.5, 78.1)
- added C1004: 100nF, Capacitor_SMD:C_0603_1608Metric_Pad1.08x0.95mm_HandSolder, F.Cu at (-220.5, 80.6)
- added C1005: 100nF, Capacitor_SMD:C_0603_1608Metric_Pad1.08x0.95mm_HandSolder, F.Cu at (-220.5, 83.1)
- added C1006: 6pF, Capacitor_SMD:C_0603_1608Metric_Pad1.08x0.95mm_HandSolder, F.Cu at (-220.5, 85.7)
- added C1007: 100nF, Capacitor_SMD:C_0603_1608Metric_Pad1.08x0.95mm_HandSolder, F.Cu at (-220.5, 88.2)
- added C1008: 100nF, Capacitor_SMD:C_0603_1608Metric_Pad1.08x0.95mm_HandSolder, F.Cu at (-216.1, 73.1)
- added C1009: 100nF, Capacitor_SMD:C_0603_1608Metric_Pad1.08x0.95mm_HandSolder, F.Cu at (-216.1, 75.6)
- added C1010: 100nF, Capacitor_SMD:C_0603_1608Metric_Pad1.08x0.95mm_HandSolder, F.Cu at (-216.1, 78.1)
- added C1011: 1uF, Capacitor_SMD:C_0603_1608Metric_Pad1.08x0.95mm_HandSolder, F.Cu at (-216.1, 80.6)
- added C1012: 1uF, Capacitor_SMD:C_0603_1608Metric_Pad1.08x0.95mm_HandSolder, F.Cu at (-216.1, 83.1)
- added C1013: 1uF, Capacitor_SMD:C_0603_1608Metric_Pad1.08x0.95mm_HandSolder, F.Cu at (-216.1, 85.7)
- added C2001: 4.7nF, Capacitor_SMD:C_0603_1608Metric_Pad1.08x0.95mm_HandSolder, F.Cu at (-220.5, 95.3)
- added C2002: 100nF, Capacitor_SMD:C_0603_1608Metric_Pad1.08x0.95mm_HandSolder, F.Cu at (-220.5, 97.8)
- added C2003: 100nF, Capacitor_SMD:C_0603_1608Metric_Pad1.08x0.95mm_HandSolder, F.Cu at (-220.5, 100.3)
- added C2004: 100nF, Capacitor_SMD:C_0603_1608Metric_Pad1.08x0.95mm_HandSolder, F.Cu at (-220.5, 102.8)
- added C2005: 10nF, Capacitor_SMD:C_0603_1608Metric_Pad1.08x0.95mm_HandSolder, F.Cu at (-220.5, 105.3)
- added C2006: 1uF, Capacitor_SMD:C_0603_1608Metric_Pad1.08x0.95mm_HandSolder, F.Cu at (-220.5, 107.9)
- added C204001: 100nF, Capacitor_SMD:C_0603_1608Metric_Pad1.08x0.95mm_HandSolder, F.Cu at (-138.0, 46.0)
- added C204002: 10uF, Capacitor_SMD:C_0603_1608Metric_Pad1.08x0.95mm_HandSolder, F.Cu at (-138.0, 48.5)
- added C207001: 4.7nF, Capacitor_SMD:C_0603_1608Metric_Pad1.08x0.95mm_HandSolder, F.Cu at (-220.5, 119.6)
- added C207002: 100nF, Capacitor_SMD:C_0603_1608Metric_Pad1.08x0.95mm_HandSolder, F.Cu at (-220.5, 122.1)
- added C207003: 100nF, Capacitor_SMD:C_0603_1608Metric_Pad1.08x0.95mm_HandSolder, F.Cu at (-220.5, 124.6)
- added C207004: 100nF, Capacitor_SMD:C_0603_1608Metric_Pad1.08x0.95mm_HandSolder, F.Cu at (-220.5, 127.2)
- added C207005: 10nF, Capacitor_SMD:C_0603_1608Metric_Pad1.08x0.95mm_HandSolder, F.Cu at (-220.5, 129.7)
- added C207006: 1uF, Capacitor_SMD:C_0603_1608Metric_Pad1.08x0.95mm_HandSolder, F.Cu at (-220.5, 132.2)
- added C208001: 4.7nF, Capacitor_SMD:C_0603_1608Metric_Pad1.08x0.95mm_HandSolder, F.Cu at (-174.0, 46.0)
- added C208002: 100nF, Capacitor_SMD:C_0603_1608Metric_Pad1.08x0.95mm_HandSolder, F.Cu at (-174.0, 48.5)
- added C208003: 100nF, Capacitor_SMD:C_0603_1608Metric_Pad1.08x0.95mm_HandSolder, F.Cu at (-174.0, 51.0)
- added C208004: 100nF, Capacitor_SMD:C_0603_1608Metric_Pad1.08x0.95mm_HandSolder, F.Cu at (-174.0, 53.5)
- added C208005: 10nF, Capacitor_SMD:C_0603_1608Metric_Pad1.08x0.95mm_HandSolder, F.Cu at (-174.0, 56.0)
- added C208006: 1uF, Capacitor_SMD:C_0603_1608Metric_Pad1.08x0.95mm_HandSolder, F.Cu at (-174.0, 58.5)
- added C4001: 100nF, Capacitor_SMD:C_0603_1608Metric_Pad1.08x0.95mm_HandSolder, F.Cu at (-120.2, 46.0)
- added C4002: 10uF, Capacitor_SMD:C_0603_1608Metric_Pad1.08x0.95mm_HandSolder, F.Cu at (-120.2, 48.5)
- added C5001: 100nF, Capacitor_SMD:C_0603_1608Metric_Pad1.08x0.95mm_HandSolder, F.Cu at (-174.0, 70.3)
- added C5002: 10uF, Capacitor_SMD:C_0603_1608Metric_Pad1.08x0.95mm_HandSolder, F.Cu at (-174.0, 72.8)
- added C5003: 10uF, Capacitor_SMD:C_0603_1608Metric_Pad1.08x0.95mm_HandSolder, F.Cu at (-174.0, 75.3)
- added C5004: 10uF, Capacitor_SMD:C_0603_1608Metric_Pad1.08x0.95mm_HandSolder, F.Cu at (-174.0, 77.8)
- added C5005: 10uF, Capacitor_SMD:C_0603_1608Metric_Pad1.08x0.95mm_HandSolder, F.Cu at (-174.0, 80.3)
- added C_LED107001: 100nF, Capacitor_SMD:C_0603_1608Metric_Pad1.08x0.95mm_HandSolder, B.Cu at (63.7, 124.3)
- added C_LED108001: 100nF, Capacitor_SMD:C_0603_1608Metric_Pad1.08x0.95mm_HandSolder, B.Cu at (63.7, 105.2)
- added C_LED109001: 100nF, Capacitor_SMD:C_0603_1608Metric_Pad1.08x0.95mm_HandSolder, B.Cu at (63.7, 86.2)
- added C_LED110001: 100nF, Capacitor_SMD:C_0603_1608Metric_Pad1.08x0.95mm_HandSolder, B.Cu at (82.7, 110.3)
- added C_LED111001: 100nF, Capacitor_SMD:C_0603_1608Metric_Pad1.08x0.95mm_HandSolder, B.Cu at (82.7, 91.2)
- added C_LED112001: 100nF, Capacitor_SMD:C_0603_1608Metric_Pad1.08x0.95mm_HandSolder, B.Cu at (82.7, 72.2)
- added C_LED113001: 100nF, Capacitor_SMD:C_0603_1608Metric_Pad1.08x0.95mm_HandSolder, B.Cu at (101.7, 100.3)
- added C_LED114001: 100nF, Capacitor_SMD:C_0603_1608Metric_Pad1.08x0.95mm_HandSolder, B.Cu at (101.7, 81.2)
- added C_LED115001: 100nF, Capacitor_SMD:C_0603_1608Metric_Pad1.08x0.95mm_HandSolder, B.Cu at (101.7, 62.2)
- added C_LED116001: 100nF, Capacitor_SMD:C_0603_1608Metric_Pad1.08x0.95mm_HandSolder, B.Cu at (120.7, 107.3)
- added C_LED117001: 100nF, Capacitor_SMD:C_0603_1608Metric_Pad1.08x0.95mm_HandSolder, B.Cu at (120.7, 88.2)
- added C_LED118001: 100nF, Capacitor_SMD:C_0603_1608Metric_Pad1.08x0.95mm_HandSolder, B.Cu at (120.7, 69.2)
- added C_LED119001: 100nF, Capacitor_SMD:C_0603_1608Metric_Pad1.08x0.95mm_HandSolder, B.Cu at (139.7, 111.3)
- added C_LED120001: 100nF, Capacitor_SMD:C_0603_1608Metric_Pad1.08x0.95mm_HandSolder, B.Cu at (139.7, 92.2)
- added C_LED121001: 100nF, Capacitor_SMD:C_0603_1608Metric_Pad1.08x0.95mm_HandSolder, B.Cu at (139.7, 73.2)
- added C_LED122001: 100nF, Capacitor_SMD:C_0603_1608Metric_Pad1.08x0.95mm_HandSolder, B.Cu at (158.7, 149.4)
- added C_LED123001: 100nF, Capacitor_SMD:C_0603_1608Metric_Pad1.08x0.95mm_HandSolder, B.Cu at (234.7, 124.3)
- added C_LED124001: 100nF, Capacitor_SMD:C_0603_1608Metric_Pad1.08x0.95mm_HandSolder, B.Cu at (234.7, 105.2)
- added C_LED125001: 100nF, Capacitor_SMD:C_0603_1608Metric_Pad1.08x0.95mm_HandSolder, B.Cu at (234.7, 86.2)
- added C_LED126001: 100nF, Capacitor_SMD:C_0603_1608Metric_Pad1.08x0.95mm_HandSolder, B.Cu at (215.7, 110.3)
- added C_LED127001: 100nF, Capacitor_SMD:C_0603_1608Metric_Pad1.08x0.95mm_HandSolder, B.Cu at (215.7, 91.2)
- added C_LED128001: 100nF, Capacitor_SMD:C_0603_1608Metric_Pad1.08x0.95mm_HandSolder, B.Cu at (215.7, 72.2)
- added C_LED129001: 100nF, Capacitor_SMD:C_0603_1608Metric_Pad1.08x0.95mm_HandSolder, B.Cu at (196.7, 100.3)
- added C_LED130001: 100nF, Capacitor_SMD:C_0603_1608Metric_Pad1.08x0.95mm_HandSolder, B.Cu at (196.7, 81.2)
- added C_LED131001: 100nF, Capacitor_SMD:C_0603_1608Metric_Pad1.08x0.95mm_HandSolder, B.Cu at (196.7, 62.2)
- added C_LED132001: 100nF, Capacitor_SMD:C_0603_1608Metric_Pad1.08x0.95mm_HandSolder, B.Cu at (177.7, 107.3)
- added C_LED133001: 100nF, Capacitor_SMD:C_0603_1608Metric_Pad1.08x0.95mm_HandSolder, B.Cu at (177.7, 88.2)
- added C_LED134001: 100nF, Capacitor_SMD:C_0603_1608Metric_Pad1.08x0.95mm_HandSolder, B.Cu at (177.7, 69.2)
- added C_LED135001: 100nF, Capacitor_SMD:C_0603_1608Metric_Pad1.08x0.95mm_HandSolder, B.Cu at (158.7, 111.3)
- added C_LED136001: 100nF, Capacitor_SMD:C_0603_1608Metric_Pad1.08x0.95mm_HandSolder, B.Cu at (158.7, 92.2)
- added C_LED137001: 100nF, Capacitor_SMD:C_0603_1608Metric_Pad1.08x0.95mm_HandSolder, B.Cu at (158.7, 73.2)
- added C_LED138001: 100nF, Capacitor_SMD:C_0603_1608Metric_Pad1.08x0.95mm_HandSolder, B.Cu at (139.7, 149.4)
- added C_TMR10001: 100nF, Capacitor_SMD:C_0603_1608Metric_Pad1.08x0.95mm_HandSolder, B.Cu at (77.7, 102.3)
- added C_TMR11001: 100nF, Capacitor_SMD:C_0603_1608Metric_Pad1.08x0.95mm_HandSolder, B.Cu at (77.7, 83.2)
- added C_TMR12001: 100nF, Capacitor_SMD:C_0603_1608Metric_Pad1.08x0.95mm_HandSolder, B.Cu at (77.7, 64.2)
- added C_TMR13001: 100nF, Capacitor_SMD:C_0603_1608Metric_Pad1.08x0.95mm_HandSolder, B.Cu at (96.7, 92.3)
- added C_TMR14001: 100nF, Capacitor_SMD:C_0603_1608Metric_Pad1.08x0.95mm_HandSolder, B.Cu at (96.7, 73.2)
- added C_TMR15001: 100nF, Capacitor_SMD:C_0603_1608Metric_Pad1.08x0.95mm_HandSolder, B.Cu at (96.7, 54.2)
- added C_TMR16001: 100nF, Capacitor_SMD:C_0603_1608Metric_Pad1.08x0.95mm_HandSolder, B.Cu at (115.7, 99.3)
- added C_TMR17001: 100nF, Capacitor_SMD:C_0603_1608Metric_Pad1.08x0.95mm_HandSolder, B.Cu at (115.7, 80.2)
- added C_TMR18001: 100nF, Capacitor_SMD:C_0603_1608Metric_Pad1.08x0.95mm_HandSolder, B.Cu at (115.7, 61.2)
- added C_TMR19001: 100nF, Capacitor_SMD:C_0603_1608Metric_Pad1.08x0.95mm_HandSolder, B.Cu at (134.7, 103.3)
- added C_TMR20001: 100nF, Capacitor_SMD:C_0603_1608Metric_Pad1.08x0.95mm_HandSolder, B.Cu at (134.7, 84.2)
- added C_TMR21001: 100nF, Capacitor_SMD:C_0603_1608Metric_Pad1.08x0.95mm_HandSolder, B.Cu at (134.7, 65.2)
- added C_TMR22001: 100nF, Capacitor_SMD:C_0603_1608Metric_Pad1.08x0.95mm_HandSolder, B.Cu at (153.7, 141.4)
- added C_TMR23001: 100nF, Capacitor_SMD:C_0603_1608Metric_Pad1.08x0.95mm_HandSolder, B.Cu at (229.7, 116.3)
- added C_TMR24001: 100nF, Capacitor_SMD:C_0603_1608Metric_Pad1.08x0.95mm_HandSolder, B.Cu at (229.7, 97.2)
- added C_TMR25001: 100nF, Capacitor_SMD:C_0603_1608Metric_Pad1.08x0.95mm_HandSolder, B.Cu at (229.7, 78.2)
- added C_TMR26001: 100nF, Capacitor_SMD:C_0603_1608Metric_Pad1.08x0.95mm_HandSolder, B.Cu at (210.7, 102.3)
- added C_TMR27001: 100nF, Capacitor_SMD:C_0603_1608Metric_Pad1.08x0.95mm_HandSolder, B.Cu at (210.7, 83.2)
- added C_TMR28001: 100nF, Capacitor_SMD:C_0603_1608Metric_Pad1.08x0.95mm_HandSolder, B.Cu at (210.7, 64.2)
- added C_TMR29001: 100nF, Capacitor_SMD:C_0603_1608Metric_Pad1.08x0.95mm_HandSolder, B.Cu at (191.7, 92.3)
- added C_TMR30001: 100nF, Capacitor_SMD:C_0603_1608Metric_Pad1.08x0.95mm_HandSolder, B.Cu at (191.7, 73.2)
- added C_TMR31001: 100nF, Capacitor_SMD:C_0603_1608Metric_Pad1.08x0.95mm_HandSolder, B.Cu at (191.7, 54.2)
- added C_TMR32001: 100nF, Capacitor_SMD:C_0603_1608Metric_Pad1.08x0.95mm_HandSolder, B.Cu at (172.7, 99.3)
- added C_TMR33001: 100nF, Capacitor_SMD:C_0603_1608Metric_Pad1.08x0.95mm_HandSolder, B.Cu at (172.7, 80.2)
- added C_TMR34001: 100nF, Capacitor_SMD:C_0603_1608Metric_Pad1.08x0.95mm_HandSolder, B.Cu at (172.7, 61.2)
- added C_TMR35001: 100nF, Capacitor_SMD:C_0603_1608Metric_Pad1.08x0.95mm_HandSolder, B.Cu at (153.7, 103.3)
- added C_TMR36001: 100nF, Capacitor_SMD:C_0603_1608Metric_Pad1.08x0.95mm_HandSolder, B.Cu at (153.7, 84.2)
- added C_TMR37001: 100nF, Capacitor_SMD:C_0603_1608Metric_Pad1.08x0.95mm_HandSolder, B.Cu at (153.7, 65.2)
- added C_TMR38001: 100nF, Capacitor_SMD:C_0603_1608Metric_Pad1.08x0.95mm_HandSolder, B.Cu at (134.7, 141.4)
- added C_TMR7001: 100nF, Capacitor_SMD:C_0603_1608Metric_Pad1.08x0.95mm_HandSolder, B.Cu at (58.7, 116.3)
- added C_TMR8001: 100nF, Capacitor_SMD:C_0603_1608Metric_Pad1.08x0.95mm_HandSolder, B.Cu at (58.7, 97.2)
- added C_TMR9001: 100nF, Capacitor_SMD:C_0603_1608Metric_Pad1.08x0.95mm_HandSolder, B.Cu at (58.7, 78.2)
- added D1001: D_Schottky, CUHS20S30:CUHS20S40H3F, F.Cu at (-196.1, 85.0)
- added D2001: D_Schottky, CUHS20S30:CUHS20S40H3F, F.Cu at (-203.1, 107.2)
- added D207001: D_Schottky, CUHS20S30:CUHS20S40H3F, F.Cu at (-203.1, 131.5)
- added D208001: D_Schottky, CUHS20S30:CUHS20S40H3F, F.Cu at (-156.6, 57.9)
- added FB1001: 120R, BLM21PG121SN1D:BLM21AG102BH1J, F.Cu at (-197.2, 89.4)
- added FB2001: 120R, BLM21PG121SN1D:BLM21AG102BH1J, F.Cu at (-204.2, 111.6)
- added FB207001: 120R, BLM21PG121SN1D:BLM21AG102BH1J, F.Cu at (-204.2, 135.9)
- added FB208001: 120R, BLM21PG121SN1D:BLM21AG102BH1J, F.Cu at (-157.7, 62.3)
- added IC1001: LD39100PU33RY, LD39100PU33RY:SON95P300X300X90-7N-D, F.Cu at (-182.9, 86.8)
- added IC204001: ADG726BSUZ, ADG726BSUZ:QFP50P900X900X120-48N, F.Cu at (190.8, 111.4)
- added IC4001: ADG726BSUZ, ADG726BSUZ:QFP50P900X900X120-48N, F.Cu at (97.6, 111.9)
- added IC5001: SN74AHCT1G125DBVR, SN74AHCT1G125DBVR:SOT95P280X145-5N, F.Cu at (-169.2, 71.3)
- added J1001: Conn_01x16_Socket, Connector_JST:JST_XH_S16B-XH-A_1x16_P2.50mm_Horizontal, F.Cu at (-219.2, 48.1)
- added J1002: GSB1C4621DS1HR, GSB1C4621DS1HR:GSB1C4621DS1HR, F.Cu at (-131.8, 36.3)
- added J1003: Conn_01x16_Socket, Connector_JST:JST_XH_S16B-XH-A_1x16_P2.50mm_Horizontal, F.Cu at (-219.2, 61.6)
- added J1004: TC2050, Connector:Tag-Connect_TC2050-IDC-NL_2x05_P1.27mm_Vertical, F.Cu at (-187.0, 81.6)
- added J2001: GSB1C4621DS1HR, GSB1C4621DS1HR:GSB1C4621DS1HR, F.Cu at (-169.9, 36.3)
- added J207001: GSB1C4621DS1HR, GSB1C4621DS1HR:GSB1C4621DS1HR, F.Cu at (-209.9, 123.8)
- added J208001: GSB1C4621DS1HR, GSB1C4621DS1HR:GSB1C4621DS1HR, F.Cu at (-153.3, 36.3)
- added LED107001: SK6812MINI-E, kicad-keyboard-parts:MX_SK6812MINI-E_REV, B.Cu at (58.7, 119.3)
- added LED108001: SK6812MINI-E, kicad-keyboard-parts:MX_SK6812MINI-E_REV, B.Cu at (58.7, 100.2)
- added LED109001: SK6812MINI-E, kicad-keyboard-parts:MX_SK6812MINI-E_REV, B.Cu at (58.7, 81.2)
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Other:
- board size 244.1 x 133.4 mm -> 244.1 x 133.3 mm

Commit message: [ADD](PCB) usbs and uc placement
Parts:
- moved J1003 468.3 mm to (246.9, 107.8), turned to 76 degrees
- moved C1011 434.4 mm to (213.9, 142.1), turned to -90 degrees
- moved C1009 430.9 mm to (210.2, 138.0)
- moved C1010 430.8 mm to (210.2, 139.6)
- moved C1004 424.7 mm to (200.1, 139.8), turned to -90 degrees
- moved C1007 422.0 mm to (199.5, 129.2), turned to 90 degrees
- moved C1002 421.8 mm to (197.9, 129.2), turned to 90 degrees
- moved C1008 421.0 mm to (201.1, 129.2), turned to 90 degrees
- moved R1002 420.3 mm to (205.4, 124.4), turned to -90 degrees
- moved C1005 419.3 mm to (196.3, 129.2), turned to 90 degrees
- moved C1001 419.0 mm to (194.7, 129.2), turned to 90 degrees
- moved U1002 413.2 mm to (206.1, 133.0)
- moved FB1001 411.4 mm to (210.8, 142.1), turned to 180 degrees
- moved Y1001 389.6 mm to (197.8, 134.4), turned to 90 degrees
- moved R207001 377.9 mm to (145.8, 41.6), turned to 90 degrees
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Connections:
- TMR22001 pad 1: /keys/key_bank2/S16A -> /keys/key_bank3/S16A
- TMR22001 pad 3: /keys/key_bank2/S16B -> /keys/key_bank3/S16B
- TMR38001 pad 1: /keys/key_bank3/S16A -> /keys/key_bank2/S16A
- TMR38001 pad 3: /keys/key_bank3/S16B -> /keys/key_bank2/S16B

Commit message: [ADD](Mountinghole)
Parts:
- removed C5002, C5003, C5004, C5005: 10uF, Capacitor_SMD:C_0603_1608Metric_Pad1.08x0.95mm_HandSolder
- added _1: , MountingHole_2.2mm_M2_Pad_Via, F.Cu at (40.0, 63.7)
- added _2: , MountingHole_2.2mm_M2_Pad_Via, F.Cu at (249.1, 63.7)
- added _3: , MountingHole_2.2mm_M2_Pad_Via, F.Cu at (178.8, 48.6)
- added _4: , MountingHole_2.2mm_M2_Pad_Via, F.Cu at (110.3, 48.6)
- added _5: , MountingHole_2.2mm_M2_Pad_Via, F.Cu at (121.7, 113.4)
- added _6: , MountingHole_2.2mm_M2_Pad_Via, F.Cu at (167.3, 113.4)
- added _7: , MountingHole_2.2mm_M2_Pad_Via, F.Cu at (77.8, 142.2)
- added _8: , MountingHole_2.2mm_M2_Pad_Via, F.Cu at (211.2, 142.2)
- moved R1003 447.1 mm to (235.1, 62.3), turned to 71.36 degrees
- moved R1004 445.5 mm to (233.4, 61.7), turned to 71.36 degrees
- moved D1001 424.3 mm to (227.4, 59.0), turned to 161.36 degrees
- moved C1012 421.6 mm to (203.0, 128.7)
- moved C1013 420.6 mm to (202.7, 124.2)
- moved R1005 413.3 mm to (199.2, 124.2)
- moved C1006 399.8 mm to (176.2, 134.8), turned to 90 degrees
- moved C1003 394.6 mm to (170.3, 132.3), turned to 90 degrees
- moved J1004 344.1 mm to (173.3, 148.6), turned to 180 degrees
- moved R204001 336.1 mm to (191.6, 116.2), turned to -90 degrees
- moved C204001 332.8 mm to (187.5, 115.3)
- moved C204002 332.7 mm to (187.5, 116.9)
- moved R1001 322.5 mm to (101.7, 142.3)
- moved U1001 279.0 mm to (108.6, 141.6)
- moved C5001 247.3 mm to (65.5, 131.6), turned to 180 degrees
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Connections:
- J1001 pad 10: GND -> /D1
- J1003 pad 10: GND -> /D2
- U1002 pad 12: unconnected-(U1002-PA2-Pad12) -> /nWR
- U1002 pad 13: /nWR -> /D1
- U1002 pad 14: unconnected-(U1002-PA4-Pad14) -> /D2
Routing:
- added copper zone on In2.Cu, net +3.3VA
- added copper zone on In1.Cu, net GND

Commit message: [ADD](no clue)
Parts:
- moved R1001 66.0 mm to (167.7, 143.4), turned to 180 degrees
- moved R1002 56.0 mm to (128.4, 132.1), turned to 0 degrees
- moved C_LED113001 51.6 mm to (95.0, 47.0), turned to 0 degrees
- moved C_LED129001 51.6 mm to (190.1, 47.0), turned to 0 degrees
- moved U1001 51.0 mm to (159.5, 144.1), turned to 180 degrees
- moved C1011 49.8 mm to (142.9, 147.6), turned to 45 degrees
- moved FB1001 49.8 mm to (139.7, 146.4), turned to 135 degrees
- moved C1010 47.9 mm to (141.0, 144.2), turned to -45 degrees
- moved C1009 46.8 mm to (142.1, 143.1), turned to -45 degrees
- moved C1004 45.7 mm to (133.9, 146.4), turned to -135 degrees
- moved C1001 42.7 mm to (130.9, 135.1)
- moved C1008 42.7 mm to (137.3, 135.1)
- moved C1002 42.7 mm to (134.1, 135.1)
- moved C1005 42.7 mm to (132.5, 135.1)
- moved C1007 42.7 mm to (135.7, 135.1)
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Connections:
- net /keys/key_bank2/S10A renamed /keys/key_bank2/S10+
- net /keys/key_bank2/S10B renamed /keys/key_bank2/S10-
- net /keys/key_bank2/S11A renamed /keys/key_bank2/S11+
- net /keys/key_bank2/S11B renamed /keys/key_bank2/S11-
- net /keys/key_bank2/S12A renamed /keys/key_bank2/S12+
- net /keys/key_bank2/S12B renamed /keys/key_bank2/S12-
- net /keys/key_bank2/S13A renamed /keys/key_bank2/S13+
- net /keys/key_bank2/S13B renamed /keys/key_bank2/S13-
- net /keys/key_bank2/S14A renamed /keys/key_bank2/S14+
- net /keys/key_bank2/S14B renamed /keys/key_bank2/S14-
- net /keys/key_bank2/S15A renamed /keys/key_bank2/S15+
- net /keys/key_bank2/S15B renamed /keys/key_bank2/S15-
- net /keys/key_bank2/S16A renamed /keys/key_bank2/S16+
- net /keys/key_bank2/S16B renamed /keys/key_bank2/S16-
- net /keys/key_bank2/S1A renamed /keys/key_bank2/S1+
- net /keys/key_bank2/S1B renamed /keys/key_bank2/S1-
- net /keys/key_bank2/S2A renamed /keys/key_bank2/S2+
- net /keys/key_bank2/S2B renamed /keys/key_bank2/S2-
- net /keys/key_bank2/S3A renamed /keys/key_bank2/S3+
- net /keys/key_bank2/S3B renamed /keys/key_bank2/S3-
- net /keys/key_bank2/S4A renamed /keys/key_bank2/S4+
- net /keys/key_bank2/S4B renamed /keys/key_bank2/S4-
- net /keys/key_bank2/S5A renamed /keys/key_bank2/S5+
- net /keys/key_bank2/S5B renamed /keys/key_bank2/S5-
- net /keys/key_bank2/S6A renamed /keys/key_bank2/S6+
- net /keys/key_bank2/S6B renamed /keys/key_bank2/S6-
- net /keys/key_bank2/S7A renamed /keys/key_bank2/S7+
- net /keys/key_bank2/S7B renamed /keys/key_bank2/S7-
- net /keys/key_bank2/S8A renamed /keys/key_bank2/S8+
- net /keys/key_bank2/S8B renamed /keys/key_bank2/S8-
- net /keys/key_bank2/S9A renamed /keys/key_bank2/S9+
- net /keys/key_bank2/S9B renamed /keys/key_bank2/S9-
- net /keys/key_bank3/S10A renamed /keys/key_bank3/S10+
- net /keys/key_bank3/S10B renamed /keys/key_bank3/S10-
- net /keys/key_bank3/S11A renamed /keys/key_bank3/S11+
- net /keys/key_bank3/S11B renamed /keys/key_bank3/S11-
- net /keys/key_bank3/S12A renamed /keys/key_bank3/S12+
- net /keys/key_bank3/S12B renamed /keys/key_bank3/S12-
- net /keys/key_bank3/S13A renamed /keys/key_bank3/S13+
- net /keys/key_bank3/S13B renamed /keys/key_bank3/S13-
- net /keys/key_bank3/S14A renamed /keys/key_bank3/S14+
- net /keys/key_bank3/S14B renamed /keys/key_bank3/S14-
- net /keys/key_bank3/S15A renamed /keys/key_bank3/S15+
- net /keys/key_bank3/S15B renamed /keys/key_bank3/S15-
- net /keys/key_bank3/S16A renamed /keys/key_bank3/S16+
- net /keys/key_bank3/S16B renamed /keys/key_bank3/S16-
- net /keys/key_bank3/S1A renamed /keys/key_bank3/S1+
- net /keys/key_bank3/S1B renamed /keys/key_bank3/S1-
- net /keys/key_bank3/S2A renamed /keys/key_bank3/S2+
- net /keys/key_bank3/S2B renamed /keys/key_bank3/S2-
- net /keys/key_bank3/S3A renamed /keys/key_bank3/S3+
- net /keys/key_bank3/S3B renamed /keys/key_bank3/S3-
- net /keys/key_bank3/S4A renamed /keys/key_bank3/S4+
- net /keys/key_bank3/S4B renamed /keys/key_bank3/S4-
- net /keys/key_bank3/S5A renamed /keys/key_bank3/S5+
- net /keys/key_bank3/S5B renamed /keys/key_bank3/S5-
- net /keys/key_bank3/S6A renamed /keys/key_bank3/S6+
- net /keys/key_bank3/S6B renamed /keys/key_bank3/S6-
- net /keys/key_bank3/S7A renamed /keys/key_bank3/S7+
- net /keys/key_bank3/S7B renamed /keys/key_bank3/S7-
- net /keys/key_bank3/S8A renamed /keys/key_bank3/S8+
- net /keys/key_bank3/S8B renamed /keys/key_bank3/S8-
- net /keys/key_bank3/S9A renamed /keys/key_bank3/S9+
- net /keys/key_bank3/S9B renamed /keys/key_bank3/S9-
- D1001 pad 1: Net-(D1001-K) -> VBUS
- J1002 pad A4: Net-(D1001-K) -> VBUS
- J1002 pad A9: Net-(D1001-K) -> VBUS
- LED114001 pad 2: /LEDs/LED16/DIN -> /LEDs/LED7/DOUT
- LED115001 pad 4: /LEDs/LED23/DOUT -> /LEDs/LED7/DOUT
- LED123001 pad 4: /LEDs/LED16/DIN -> /LEDs/LED15/DOUT
- LED131001 pad 4: /LEDs/LED15/DOUT -> /LEDs/LED23/DOUT
- U1002 pad 18: /A0 -> /A3
- U1002 pad 19: /A1 -> /A2
- U1002 pad 20: /A2 -> /A1
- U1002 pad 21: /A3 -> /A0
- U1002 pad 25: /CS_USB3 -> /nCS_FLASH
- U1002 pad 27: /CS_USB1 -> /CS_USB3
- U1002 pad 28: /nCS_FLASH -> /CS_USB1
- U1002 pad 39: /nCS0 -> /nCS5
- U1002 pad 40: /nCS1 -> /nCS4
- U1002 pad 41: /nCS2 -> /nCS1
- U1002 pad 42: /nCS3 -> /nCS0
- U1002 pad 43: /nCS4 -> /nCS3
- U1002 pad 45: /nCS5 -> /nCS2
Routing:
- net GND: track 0.00 -> 194.3 mm, vias 0 -> 105
- net /SPI1_MISO: track 0.00 -> 193.2 mm, vias 0 -> 5
- net /SPI1_CLK: track 0.00 -> 167.7 mm, vias 0 -> 4
- net /USB+: track 0.00 -> 166.2 mm, vias 0 -> 4
- net /USB-: track 0.00 -> 163.8 mm, vias 0 -> 2
- net /SPI1_MOSI: track 0.00 -> 163.4 mm, vias 0 -> 5
- net /nCS3: track 0.00 -> 149.7 mm, vias 0 -> 1
- net /DA+: track 0.00 -> 148.9 mm, vias 0 -> 3
- net /nCS2: track 0.00 -> 148.6 mm, vias 0 -> 1
- net /DA-: track 0.00 -> 147.3 mm, vias 0 -> 3
- net /A0: track 0.00 -> 139.8 mm, vias 0 -> 2
- net /A1: track 0.00 -> 137.9 mm, vias 0 -> 2
- net /A2: track 0.00 -> 135.8 mm, vias 0 -> 2
- net /A3: track 0.00 -> 133.8 mm, vias 0 -> 2
- net /nWR: track 0.00 -> 129.4 mm, vias 0 -> 2
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- added copper zone on In2.Cu, net GND
- removed copper zone on In2.Cu, net +3.3VA
Other:
- board size 244.1 x 133.3 mm -> 244.1 x 123.8 mm
