File: key_bank.kicad_sch (KiCad schematic)
At the start: 4 parts, among them IC4001 ADG726BSUZ

Commit message: [ADD](no clue)
Connections:
- net S10A renamed S10+
- net S10B renamed S10-
- net S11A renamed S11+
- net S11B renamed S11-
- net S12A renamed S12+
- net S12B renamed S12-
- net S13A renamed S13+
- net S13B renamed S13-
- net S14A renamed S14+
- net S14B renamed S14-
- net S15A renamed S15+
- net S15B renamed S15-
- net S16A renamed S16+
- net S16B renamed S16-
- net S1A renamed S1+
- net S1B renamed S1-
- net S2A renamed S2+
- net S2B renamed S2-
- net S3A renamed S3+
- net S3B renamed S3-
- net S4A renamed S4+
- net S4B renamed S4-
- net S5A renamed S5+
- net S5B renamed S5-
- net S6A renamed S6+
- net S6B renamed S6-
- net S7A renamed S7+
- net S7B renamed S7-
- net S8A renamed S8+
- net S8B renamed S8-
- net S9A renamed S9+
- net S9B renamed S9-
Changed lines of the file:
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@@
 		)
 	)
-	(label "S13A"
+	(label "S13+"
 		(at 137.16 114.3 180)
 		(effects
@@
 		)
 	)
-	(label "S4B"
+	(label "S4-"
 		(at 175.26 78.74 90)
 		(effects
@@
 		)
 	)
-	(label "S11B"
+	(label "S11-"
 		(at 77.47 135.89 0)
 		(effects
@@
 		)
 	)
-	(label "S14B"
+	(label "S14-"
 		(at 77.47 166.37 0)
 		(effects
@@
 		)
 	)
-	(label "S5A"
+	(label "S5+"
 		(at 77.47 72.39 0)
 		(effects
@@
 		)
 	)
-	(label "S8B"
+	(label "S8-"
 		(at 165.1 78.74 90)
 		(effects
@@
 		)
 	)
-	(label "S3B"
+	(label "S3-"
 		(at 77.47 54.61 0)
 		(effects
@@
 		)
 	)
-	(label "S14A"
+	(label "S14+"
 		(at 137.16 111.76 180)
 		(effects
@@
 		)
 	)
-	(label "S8A"
+	(label "S8+"
 		(at 77.47 102.87 0)
 		(effects
@@
 		)
 	)
-	(label "S15B"
+	(label "S15-"
 		(at 137.16 91.44 180)
 		(effects
@@
 		)
 	)
-	(label "S12B"
+	(label "S12-"
 		(at 154.94 78.74 90)
 		(effects
@@
 		)
 	)
-	(label "S2A"
+	(label "S2+"
 		(at 77.47 41.91 0)
 		(effects
@@
 		)
 	)
-	(label "S9B"
+	(label "S9-"
 		(at 77.47 115.57 0)
 		(effects
@@
 		)
 	)
-	(label "S1A"
+	(label "S1+"
 		(at 77.47 31.75 0)
 		(effects
@@
 		)
 	)
-	(label "S12A"
+	(label "S12+"
 		(at 154.94 121.92 270)
 		(effects
@@
 		)
 	)
-	(label "S11A"
+	(label "S11+"
 		(at 157.48 121.92 270)
 		(effects
@@
 		)
 	)
-	(label "S16A"
+	(label "S16+"
 		(at 137.16 106.68 180)
 		(effects
@@
 		)
 	)
-	(label "S14B"
+	(label "S14-"
 		(at 137.16 88.9 180)
 		(effects
@@
 		)
 	)
-	(label "S6B"
+	(label "S6-"
 		(at 77.47 85.09 0)
 		(effects
@@
 		)
 	)
-	(label "S13B"
+	(label "S13-"
 		(at 137.16 86.36 180)
 		(effects
@@
 		)
 	)
-	(label "S13A"
+	(label "S13+"
 		(at 77.47 153.67 0)
 		(effects
@@
 		)
 	)
-	(label "S4A"
+	(label "S4+"
 		(at 175.26 121.92 270)
 		(effects
@@
 		)
 	)
-	(label "S9A"
+	(label "S9+"
 		(at 77.47 113.03 0)
 		(effects
@@
 		)
 	)
-	(label "S6A"
+	(label "S6+"
 		(at 170.18 121.92 270)
 		(effects
@@
 		)
 	)
-	(label "S13B"
+	(label "S13-"
 		(at 77.47 156.21 0)
 		(effects
@@
 		)
 	)
-	(label "S10B"
+	(label "S10-"
 		(at 160.02 78.74 90)
 		(effects
@@
 		)
 	)
-	(label "S9B"
+	(label "S9-"
 		(at 162.56 78.74 90)
 		(effects
@@
 		)
 	)
-	(label "S5B"
+	(label "S5-"
 		(at 172.72 78.74 90)
 		(effects
@@
 		)
 	)
-	(label "S2A"
+	(label "S2+"
 		(at 180.34 121.92 270)
 		(effects
@@
 		)
 	)
-	(label "S10A"
+	(label "S10+"
 		(at 160.02 121.92 270)
 		(effects
@@
 		)
 	)
-	(label "S4B"
+	(label "S4-"
 		(at 77.47 64.77 0)
 		(effects
@@
 		)
 	)
-	(label "S15A"
+	(label "S15+"
 		(at 77.47 173.99 0)
 		(effects
@@
 		)
 	)
-	(label "S7A"
+	(label "S7+"
 		(at 77.47 92.71 0)
 		(effects
@@
 		)
 	)
-	(label "S3A"
+	(label "S3+"
 		(at 77.47 52.07 0)
 		(effects
@@
 		)
 	)
-	(label "S7B"
+	(label "S7-"
 		(at 77.47 95.25 0)
 		(effects
@@
 		)
 	)
-	(label "S5A"
+	(label "S5+"
 		(at 172.72 121.92 270)
 		(effects
@@
 		)
 	)
-	(label "S16A"
+	(label "S16+"
 		(at 77.47 184.15 0)
 		(effects
@@
 		)
 	)
-	(label "S7A"
+	(label "S7+"
 		(at 167.64 121.92 270)
 		(effects
@@
 		)
 	)
-	(label "S10B"
+	(label "S10-"
 		(at 77.47 125.73 0)
 		(effects
@@
 		)
 	)
-	(label "S2B"
+	(label "S2-"
 		(at 77.47 44.45 0)
 		(effects
@@
 		)
 	)
-	(label "S16B"
+	(label "S16-"
 		(at 77.47 186.69 0)
 		(effects
@@
 		)
 	)
-	(label "S14A"
+	(label "S14+"
 		(at 77.47 163.83 0)
 		(effects
@@
 		)
 	)
-	(label "S6B"
+	(label "S6-"
 		(at 170.18 78.74 90)
 		(effects
@@
 		)
 	)
-	(label "S11B"
+	(label "S11-"
 		(at 157.48 78.74 90)
 		(effects
@@
 		)
 	)
-	(label "S16B"
+	(label "S16-"
 		(at 137.16 93.98 180)
 		(effects
@@
 		)
 	)
-	(label "S12B"
+	(label "S12-"
 		(at 77.47 146.05 0)
 		(effects
@@
 		)
 	)
-	(label "S8A"
+	(label "S8+"
 		(at 165.1 121.92 270)
 		(effects
@@
 		)
 	)
-	(label "S5B"
+	(label "S5-"
 		(at 77.47 74.93 0)
 		(effects
@@
 		)
 	)
-	(label "S3B"
+	(label "S3-"
 		(at 177.8 78.74 90)
 		(effects
@@
 		)
 	)
-	(label "S6A"
+	(label "S6+"
 		(at 77.47 82.55 0)
 		(effects
@@
 		)
 	)
-	(label "S10A"
+	(label "S10+"
 		(at 77.47 123.19 0)
 		(effects
@@
 		)
 	)
-	(label "S15A"
+	(label "S15+"
 		(at 137.16 109.22 180)
 		(effects
@@
 		)
 	)
-	(label "S11A"
+	(label "S11+"
 		(at 77.47 133.35 0)
 		(effects
@@
 		)
 	)
-	(label "S1A"
+	(label "S1+"
 		(at 182.88 121.92 270)
 		(effects
@@
 		)
 	)
-	(label "S15B"
+	(label "S15-"
 		(at 77.47 176.53 0)
 		(effects
@@
 		)
 	)
-	(label "S2B"
+	(label "S2-"
 		(at 180.34 78.74 90)
 		(effects
@@
 		)
 	)
-	(label "S4A"
+	(label "S4+"
 		(at 77.47 62.23 0)
 		(effects
@@
 		)
 	)
-	(label "S3A"
+	(label "S3+"
 		(at 177.8 121.92 270)
 		(effects
@@
 		)
 	)
-	(label "S1B"
+	(label "S1-"
 		(at 77.47 34.29 0)
 		(effects
@@
 		)
 	)
-	(label "S12A"
+	(label "S12+"
 		(at 77.47 143.51 0)
 		(effects
@@
 		)
 	)
-	(label "S7B"
+	(label "S7-"
 		(at 167.64 78.74 90)
 		(effects
@@
 		)
 	)
-	(label "S1B"
+	(label "S1-"
 		(at 182.88 78.74 90)
 		(effects
@@
 		)
 	)
-	(label "S9A"
+	(label "S9+"
 		(at 162.56 121.92 270)
 		(effects
@@
 		)
 	)
-	(label "S8B"
+	(label "S8-"
 		(at 77.47 105.41 0)
 		(effects
